File: Hardware/edison_mezzanine_9dof.brd (EAGLE design)
At the start: 30.5 x 44.5 mm, 43 parts, among them U1 LSM9DS0, U2 EDISON_CONNECTOR_FULLMOUNTING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, U3 EDISON_CONNECTOR_FULLHEADER

Commit message: Fixed hanging wire from LDO and added LDO chip name to schematic.
Parts:
- U4: value (none) -> MIC52053.3V
Changed lines of the file:
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@@
 <setting verticaltext="up"/>
 </settings>
-<grid distance="0.05" unitdist="inch" unit="inch" style="dots" multiple="1" display="yes" altdistance="0.025" altunitdist="inch" altunit="inch"/>
+<grid distance="0.05" unitdist="inch" unit="inch" style="dots" multiple="1" display="yes" altdistance="0.005" altunitdist="inch" altunit="inch"/>
 <layers>
 <layer number="1" name="Top" color="4" fill="1" visible="yes" active="yes"/>
@@
 <element name="SJ2" library="SparkFun-Passives" package="PAD-JUMPER-3-NC_BY_PASTE_YES_SILK_FULL_BOX" value="JUMPER-PAD-3-NC_BY_PASTE" x="9.525" y="2.54" rot="R90"/>
 <element name="SJ1" library="SparkFun-Passives" package="PAD-JUMPER-3-NC_BY_PASTE_YES_SILK_FULL_BOX" value="JUMPER-PAD-3-NC_BY_PASTE" x="5.715" y="2.54" rot="R90"/>
-<element name="U4" library="SparkFun-PowerIC" package="SOT23-5" value="" x="9.525" y="21.59">
+<element name="U4" library="SparkFun-PowerIC" package="SOT23-5" value="MIC52053.3V" x="9.525" y="21.59">
 <attribute name="PROD_ID" value="VREG-00822" x="9.525" y="21.59" size="1.778" layer="27" font="vector" ratio="15" display="off"/>
 </element>
@@
 <contactref element="U4" pad="3"/>
 <contactref element="C1" pad="1"/>
-<contactref element="U4" pad="1"/>
 <via x="22.08" y="22.58" extent="1-16" drill="0.3302"/>
 <via x="7.62" y="21.336" extent="1-16" drill="0.3302"/>
@@
 <wire x1="6.35" y1="18.796" x2="6.35" y2="19.47" width="0.254" layer="1"/>
 <wire x1="7.874" y1="18.288" x2="9.398" y2="18.288" width="0.254" layer="1"/>
-<wire x1="8.575" y1="20.2899" x2="8.575" y2="19.497" width="0.254" layer="1"/>
 <wire x1="8.575" y1="19.497" x2="7.62" y2="18.542" width="0.254" layer="1"/>
 <wire x1="22.08" y1="22.58" x2="14.706" y2="22.58" width="0.381" layer="16"/>
@@
 <wire x1="23.32" y1="22.1798" x2="22.4802" y2="22.1798" width="0.2" layer="1"/>
 <wire x1="22.4802" y1="22.1798" x2="22.08" y2="22.58" width="0.2" layer="1"/>
+<contactref element="U4" pad="1"/>
+<wire x1="8.575" y1="20.2899" x2="8.575" y2="19.497" width="0.254" layer="1"/>
 </signal>
 <signal name="3.3V">
