File: Production Files/9dof_block-Panel-v10.brd (EAGLE design)
At the start: 30.5 x 44.5 mm, 42 parts, among them U1 LSM9DS0, U2 EDISON_CONNECTOR_FULLMOUNTING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, U3 EDISON_CONNECTOR_FULLHEADER, U4 MIC52053.3V

Commit message: moved fid
Parts:
- removed FRAME1, FRAME2: FRAME-LETTER, SparkFun-Aesthetics:CREATIVE_COMMONS
Other:
- board text removed: "NOTE: Units are in Inches"
- board text removed: "Shawn Hymel"

Commit message: created v10 panels
Parts:
- added C10, C16, C22, C28, C34, C40, C46: 10uF, SparkFun-Capacitors:0805
- added C11, C15, C17, C21, C23, C27, C29, C33, C35, C39, C41, C45, C47, C9: 1.0uF, SparkFun-Capacitors:0603-CAP
- added C12, C18, C24, C30, C36, C42, C48: 0.1uF, SparkFun-Capacitors:0603-CAP
- added C13, C19, C25, C31, C37, C43, C7: 0.22uF, SparkFun-Capacitors:0603-CAP
- added C14, C20, C26, C32, C38, C44, C8: 4.7uF, SparkFun-Capacitors:0603-CAP
- added E$1, E$2: (no value), SparkFun-Retired:FIDUCIAL-1.5X3
- added E$3, E$4, E$5, E$6: (no value), SparkFun-Aesthetics:FIDUCIAL-1X2
- added FID10, FID11, FID12, FID13, FID14, FID15, FID16, FID17, FID18, FID19, FID20, FID21, FID22, FID23, FID24, FID25, FID26, FID27, FID28, FID29, FID30, FID31, FID32, FID5, FID6, FID7, FID8, FID9: FIDUCIAL1X2, SparkFun-Aesthetics:FIDUCIAL-1X2
- added LOGO10, LOGO13, LOGO16, LOGO19, LOGO22, LOGO4, LOGO7: OSHW-LOGOS, SparkFun-Aesthetics:OSHW-LOGO-S
- added LOGO11, LOGO14, LOGO17, LOGO20, LOGO23, LOGO5, LOGO8: SFE_LOGO_NAME_FLAME.1_INCH, SparkFun-Aesthetics:SFE_LOGO_NAME_FLAME_.1
- added LOGO12, LOGO15, LOGO18, LOGO21, LOGO24, LOGO6, LOGO9: SFE_LOGO_FLAME.2_INCH, SparkFun-Aesthetics:SFE_LOGO_FLAME_.2
- added R10, R11, R12, R15, R16, R17, R18, R21, R22, R23, R24, R27, R28, R29, R30, R33, R34, R35, R36, R39, R40, R41, R42, R45, R46, R47, R48, R9: 10k, SparkFun-Resistors:0603-RES
- added R13, R14, R19, R20, R25, R26, R31, R32, R37, R38, R43, R44, R7, R8: 10K, SparkFun-Resistors:0603-RES
- added SJ100, SJ116, SJ117, SJ133, SJ134, SJ31, SJ32, SJ48, SJ49, SJ65, SJ66, SJ82, SJ83, SJ99: JUMPER-PAD-2-NC_BY_PASTE, SparkFun-Passives:PAD-JUMPER-2-NC_BY_PASTE_YES_SILK
- added SJ101, SJ102, SJ103, SJ104, SJ105, SJ106, SJ107, SJ108, SJ109, SJ110, SJ111, SJ118, SJ119, SJ120, SJ121, SJ122, SJ123, SJ124, SJ125, SJ126, SJ127, SJ128, SJ135, SJ136, SJ18, SJ19, SJ20, SJ21, SJ22, SJ23, SJ24, SJ25, SJ26, SJ33, SJ34, SJ35, SJ36, SJ37, SJ38, SJ39, SJ40, SJ41, SJ42, SJ43, SJ50, SJ51, SJ52, SJ53, SJ54, SJ55, SJ56, SJ57, SJ58, SJ59, SJ60, SJ67, SJ68, SJ69, SJ70, SJ71, SJ72, SJ73, SJ74, SJ75, SJ76, SJ77, SJ84, SJ85, SJ86, SJ87, SJ88, SJ89, SJ90, SJ91, SJ92, SJ93, SJ94: JUMPER-PAD-2-NOYES_SILK, SparkFun-Passives:PAD-JUMPER-2-NO_YES_SILK
- added SJ112, SJ113, SJ129, SJ130, SJ27, SJ28, SJ44, SJ45, SJ61, SJ62, SJ78, SJ79, SJ95, SJ96: JUMPER-PAD-3-2OF3_NC_BY_TRACE_SMALL, SparkFun-Passives:PAD-JUMPER-3-2OF3_NC_BY_TRACE_YES_SILK_FULL_BOX
- added SJ114, SJ131, SJ29, SJ46, SJ63, SJ80, SJ97: (no value), SparkFun-Passives:PAD-JUMPER-3-3OF3_NC_BY_TRACE_YES_SILK_FULL_BOX
- added SJ115, SJ132, SJ30, SJ47, SJ64, SJ81, SJ98: JUMPER-PAD-3-NOYES_SILK, SparkFun-Passives:PAD-JUMPER-3-NO_YES_SILK
- added U10, U14, U18, U22, U26, U30, U6: EDISON_CONNECTOR_FULLHEADER, Edison:DF40C-70DP-0.4(51)
- added U11, U15, U19, U23, U27, U31, U7: LSM9DS0, SparkFun-DigitalIC:LGA-24
- added U12, U16, U20, U24, U28, U32, U8: MIC52053.3V, SparkFun-PowerIC:SOT23-5
- added U13, U17, U21, U25, U29, U5, U9: EDISON_CONNECTOR_FULLMOUNTING_HOLES, Edison:EDISON_DAUGHTER
- moved C3 9.70 mm to (15.7, 32.3)
- moved SJ9 9.70 mm to (9.40, 32.3)
- moved C1 9.70 mm to (13.2, 27.2)
- moved C2 9.70 mm to (13.2, 31.0)
- moved C4 9.70 mm to (19.6, 28.4)
- moved C6 9.70 mm to (25.9, 34.8)
- moved FID1 9.70 mm to (8.13, 11.9)
- moved FID4 9.70 mm to (8.13, 11.9)
- moved LOGO3 9.70 mm to (27.9, 7.11)
- moved SJ10 9.70 mm to (27.2, 37.3)
- moved SJ12 9.70 mm to (19.6, 37.3)
- moved SJ14 9.70 mm to (11.9, 37.3)
- moved U3 9.70 mm to (31.5, 23.0)
- moved C5 9.70 mm to (22.1, 34.8)
- moved FID2 9.70 mm to (26.3, 50.0)
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Connections:
- new net 1.8V1: SJ29.2, SJ30.2, SJ31.2, SJ32.2, U5.12, U6.12, U7.18
- new net 1.8V2: SJ46.2, SJ47.2, SJ48.2, SJ49.2, U10.12, U11.18, U9.12
- new net 1.8V3: SJ63.2, SJ64.2, SJ65.2, SJ66.2, U13.12, U14.12, U15.18
- new net 1.8V4: SJ80.2, SJ81.2, SJ82.2, SJ83.2, U17.12, U18.12, U19.18
- new net 1.8V5: SJ100.2, SJ97.2, SJ98.2, SJ99.2, U21.12, U22.12, U23.18
- new net 1.8V6: SJ114.2, SJ115.2, SJ116.2, SJ117.2, U25.12, U26.12, U27.18
- new net 1.8V7: SJ131.2, SJ132.2, SJ133.2, SJ134.2, U29.12, U30.12, U31.18
- new net 3.3V1: U5.10, U5.8, U6.10, U6.8
- new net 3.3V2: U10.10, U10.8, U9.10, U9.8
- new net 3.3V3: U13.10, U13.8, U14.10, U14.8
- new net 3.3V4: U17.10, U17.8, U18.10, U18.8
- new net 3.3V5: U21.10, U21.8, U22.10, U22.8
- new net 3.3V6: U25.10, U25.8, U26.10, U26.8
- new net 3.3V7: U29.10, U29.8, U30.10, U30.8
- new net 3.3V_LOCAL1: C10.1, C12.1, C9.1, U7.15, U7.16, U7.17, U8.5
- new net 3.3V_LOCAL2: C15.1, C16.1, C18.1, U11.15, U11.16, U11.17, U12.5
- new net 3.3V_LOCAL3: C21.1, C22.1, C24.1, U15.15, U15.16, U15.17, U16.5
- new net 3.3V_LOCAL4: C27.1, C28.1, C30.1, U19.15, U19.16, U19.17, U20.5
- new net 3.3V_LOCAL5: C33.1, C34.1, C36.1, U23.15, U23.16, U23.17, U24.5
- new net 3.3V_LOCAL6: C39.1, C40.1, C42.1, U27.15, U27.16, U27.17, U28.5
- new net 3.3V_LOCAL7: C45.1, C46.1, C48.1, U31.15, U31.16, U31.17, U32.5
- new net CS_G1: R9.1, SJ18.1, U7.19
- new net CS_G2: R15.1, SJ35.1, U11.19
- new net CS_G3: R21.1, SJ52.1, U15.19
- new net CS_G4: R27.1, SJ69.1, U19.19
- new net CS_G5: R33.1, SJ86.1, U23.19
- new net CS_G6: R39.1, SJ103.1, U27.19
- new net CS_G7: R45.1, SJ120.1, U31.19
- new net CS_XM1: R10.1, SJ19.1, U7.20
- new net CS_XM2: R16.1, SJ36.1, U11.20
- new net CS_XM3: R22.1, SJ53.1, U15.20
- new net CS_XM4: R28.1, SJ70.1, U19.20
- new net CS_XM5: R34.1, SJ87.1, U23.20
- new net CS_XM6: R40.1, SJ104.1, U27.20
- new net CS_XM7: R46.1, SJ121.1, U31.20
- new net DCIN1: U5.14, U6.14
- new net DCIN2: U10.14, U9.14
- new net DCIN3: U13.14, U14.14
- new net DCIN4: U17.14, U18.14
- new net DCIN5: U21.14, U22.14
- new net DCIN6: U25.14, U26.14
- new net DCIN7: U29.14, U30.14
- new net DEN_G1: SJ22.1, U7.10
- new net DEN_G2: SJ39.1, U11.10
- new net DEN_G3: SJ56.1, U15.10
- new net DEN_G4: SJ73.1, U19.10
- new net DEN_G5: SJ90.1, U23.10
- new net DEN_G6: SJ107.1, U27.10
- new net DEN_G7: SJ124.1, U31.10
- new net DRDY_G1: SJ24.1, U7.12
- new net DRDY_G2: SJ41.1, U11.12
- new net DRDY_G3: SJ58.1, U15.12
- new net DRDY_G4: SJ75.1, U19.12
- new net DRDY_G5: SJ92.1, U23.12
- new net DRDY_G6: SJ109.1, U27.12
- new net DRDY_G7: SJ126.1, U31.12
- new net FAULT1: U5.19, U6.19
- new net FAULT2: U10.19, U9.19
- new net FAULT3: U13.19, U14.19
- new net FAULT4: U17.19, U18.19
- new net FAULT5: U21.19, U22.19
- new net FAULT6: U25.19, U26.19
- new net FAULT7: U29.19, U30.19
- new net FW_RCVR1: U5.69, U6.69
- new net FW_RCVR2: U10.69, U9.69
- new net FW_RCVR3: U13.69, U14.69
- new net FW_RCVR4: U17.69, U18.69
- new net FW_RCVR5: U21.69, U22.69
- new net FW_RCVR6: U25.69, U26.69
- new net FW_RCVR7: U29.69, U30.69
- new net GND1: C10.2, C11.2, C12.2, C8.2, C9.2, SJ33.1, SJ34.1, U5.1, U5.11, U5.13, U5.15, U5.5, U5.9, U6.1, U6.11, U6.13, U6.15, U6.5, U6.9, U7.2, U7.3, U7.4, U7.5, U7.6, U8.2
- new net GND2: C14.2, C15.2, C16.2, C17.2, C18.2, SJ50.1, SJ51.1, U10.1, U10.11, U10.13, U10.15, U10.5, U10.9, U11.2, U11.3, U11.4, U11.5, U11.6, U12.2, U9.1, U9.11, U9.13, U9.15, U9.5, U9.9
- new net GND3: C20.2, C21.2, C22.2, C23.2, C24.2, SJ67.1, SJ68.1, U13.1, U13.11, U13.13, U13.15, U13.5, U13.9, U14.1, U14.11, U14.13, U14.15, U14.5, U14.9, U15.2, U15.3, U15.4, U15.5, U15.6, U16.2
- new net GND4: C26.2, C27.2, C28.2, C29.2, C30.2, SJ84.1, SJ85.1, U17.1, U17.11, U17.13, U17.15, U17.5, U17.9, U18.1, U18.11, U18.13, U18.15, U18.5, U18.9, U19.2, U19.3, U19.4, U19.5, U19.6, U20.2
- new net GND5: C32.2, C33.2, C34.2, C35.2, C36.2, SJ101.1, SJ102.1, U21.1, U21.11, U21.13, U21.15, U21.5, U21.9, U22.1, U22.11, U22.13, U22.15, U22.5, U22.9, U23.2, U23.3, U23.4, U23.5, U23.6, U24.2
- new net GND6: C38.2, C39.2, C40.2, C41.2, C42.2, SJ118.1, SJ119.1, U25.1, U25.11, U25.13, U25.15, U25.5, U25.9, U26.1, U26.11, U26.13, U26.15, U26.5, U26.9, U27.2, U27.3, U27.4, U27.5, U27.6, U28.2
- new net GND7: C44.2, C45.2, C46.2, C47.2, C48.2, SJ135.1, SJ136.1, U29.1, U29.11, U29.13, U29.15, U29.5, U29.9, U30.1, U30.11, U30.13, U30.15, U30.5, U30.9, U31.2, U31.3, U31.4, U31.5, U31.6, U32.2
- new net GP1: U5.48, U6.48
- new net GP10: U10.48, U9.48
- new net GP109_SPI_2_CLK1: SJ28.1, U5.55, U6.55
- new net GP109_SPI_2_CLK2: SJ45.1, U10.55, U9.55
- new net GP109_SPI_2_CLK3: SJ62.1, U13.55, U14.55
- new net GP109_SPI_2_CLK4: SJ79.1, U17.55, U18.55
- new net GP109_SPI_2_CLK5: SJ96.1, U21.55, U22.55
- new net GP109_SPI_2_CLK6: SJ113.1, U25.55, U26.55
- new net GP109_SPI_2_CLK7: SJ130.1, U29.55, U30.55
- new net GP11: U10.42, U9.42
- new net GP110_SPI_2_FS1: SJ18.2, U5.53, U6.53
- new net GP110_SPI_2_FS2: SJ35.2, U10.53, U9.53
- new net GP110_SPI_2_FS3: SJ52.2, U13.53, U14.53
- new net GP110_SPI_2_FS4: SJ69.2, U17.53, U18.53
- new net GP110_SPI_2_FS5: SJ86.2, U21.53, U22.53
- new net GP110_SPI_2_FS6: SJ103.2, U25.53, U26.53
- new net GP110_SPI_2_FS7: SJ120.2, U29.53, U30.53
- new net GP111_SPI_2_FS2: SJ19.2, U5.51, U6.51
- new net GP111_SPI_2_FS3: SJ36.2, U10.51, U9.51
- new net GP111_SPI_2_FS4: SJ53.2, U13.51, U14.51
- new net GP111_SPI_2_FS5: SJ70.2, U17.51, U18.51
- new net GP111_SPI_2_FS6: SJ87.2, U21.51, U22.51
- new net GP111_SPI_2_FS7: SJ104.2, U25.51, U26.51
- new net GP111_SPI_2_FS8: SJ121.2, U29.51, U30.51
- new net GP114_SPI_2_RXD1: SJ20.2, SJ21.2, U5.59, U6.59
- new net GP114_SPI_2_RXD2: SJ37.2, SJ38.2, U10.59, U9.59
- new net GP114_SPI_2_RXD3: SJ54.2, SJ55.2, U13.59, U14.59
- new net GP114_SPI_2_RXD4: SJ71.2, SJ72.2, U17.59, U18.59
- new net GP114_SPI_2_RXD5: SJ88.2, SJ89.2, U21.59, U22.59
- new net GP114_SPI_2_RXD6: SJ105.2, SJ106.2, U25.59, U26.59
- new net GP114_SPI_2_RXD7: SJ122.2, SJ123.2, U29.59, U30.59
- new net GP115_SPI_2_TXD1: SJ27.1, U5.57, U6.57
- new net GP115_SPI_2_TXD2: SJ44.1, U10.57, U9.57
- new net GP115_SPI_2_TXD3: SJ61.1, U13.57, U14.57
- new net GP115_SPI_2_TXD4: SJ78.1, U17.57, U18.57
- new net GP115_SPI_2_TXD5: SJ95.1, U21.57, U22.57
- new net GP115_SPI_2_TXD6: SJ112.1, U25.57, U26.57
- new net GP115_SPI_2_TXD7: SJ129.1, U29.57, U30.57
- new net GP12: SJ43.2, U10.34, U9.34
- new net GP128_UART_1_CTS1: U5.65, U6.65
- new net GP128_UART_1_CTS2: U10.65, U9.65
- new net GP128_UART_1_CTS3: U13.65, U14.65
- new net GP128_UART_1_CTS4: U17.65, U18.65
- new net GP128_UART_1_CTS5: U21.65, U22.65
- new net GP128_UART_1_CTS6: U25.65, U26.65
- new net GP128_UART_1_CTS7: U29.65, U30.65
- new net GP129_UART_1_RTS1: U5.63, U6.63
- new net GP129_UART_1_RTS2: U10.63, U9.63
- new net GP129_UART_1_RTS3: U13.63, U14.63
- new net GP129_UART_1_RTS4: U17.63, U18.63
- new net GP129_UART_1_RTS5: U21.63, U22.63
- new net GP129_UART_1_RTS6: U25.63, U26.63
- new net GP129_UART_1_RTS7: U29.63, U30.63
- new net GP12_PWM1: U5.35, U6.35
- new net GP12_PWM2: U10.35, U9.35
- new net GP12_PWM3: U13.35, U14.35
- new net GP12_PWM4: U17.35, U18.35
- new net GP12_PWM5: U21.35, U22.35
- new net GP12_PWM6: U25.35, U26.35
- new net GP12_PWM7: U29.35, U30.35
- new net GP13: SJ42.2, U10.32, U9.32
- new net GP130_UART_1_RX1: U5.61, U6.61
- new net GP130_UART_1_RX2: U10.61, U9.61
- new net GP130_UART_1_RX3: U13.61, U14.61
- new net GP130_UART_1_RX4: U17.61, U18.61
- new net GP130_UART_1_RX5: U21.61, U22.61
- new net GP130_UART_1_RX6: U25.61, U26.61
- new net GP130_UART_1_RX7: U29.61, U30.61
- new net GP131_UART_1_TX1: U5.46, U6.46
- new net GP131_UART_1_TX2: U10.46, U9.46
- new net GP131_UART_1_TX3: U13.46, U14.46
- new net GP131_UART_1_TX4: U17.46, U18.46
- new net GP131_UART_1_TX5: U21.46, U22.46
- new net GP131_UART_1_TX6: U25.46, U26.46
- new net GP131_UART_1_TX7: U29.46, U30.46
- new net GP134_UART_2_RX1: U5.22, U6.22
- new net GP134_UART_2_RX2: U10.22, U9.22
- new net GP134_UART_2_RX3: U13.22, U14.22
- new net GP134_UART_2_RX4: U17.22, U18.22
- new net GP134_UART_2_RX5: U21.22, U22.22
- new net GP134_UART_2_RX6: U25.22, U26.22
- new net GP134_UART_2_RX7: U29.22, U30.22
- new net GP135_UART_2_TX1: U5.27, U6.27
- new net GP135_UART_2_TX2: U10.27, U9.27
- new net GP135_UART_2_TX3: U13.27, U14.27
- new net GP135_UART_2_TX4: U17.27, U18.27
- new net GP135_UART_2_TX5: U21.27, U22.27
- new net GP135_UART_2_TX6: U25.27, U26.27
- new net GP135_UART_2_TX7: U29.27, U30.27
- new net GP13_PWM2: U5.33, U6.33
- new net GP13_PWM3: U10.33, U9.33
- new net GP13_PWM4: U13.33, U14.33
- new net GP13_PWM5: U17.33, U18.33
- new net GP13_PWM6: U21.33, U22.33
- new net GP13_PWM7: U25.33, U26.33
- new net GP13_PWM8: U29.33, U30.33
- new net GP16: SJ41.2, U10.30, U9.30
- new net GP17: SJ40.2, U10.28, U9.28
- new net GP18: U10.26, U9.26
- new net GP182_PWM1: U5.37, U6.37
- new net GP182_PWM3: U10.37, U9.37
- new net GP182_PWM4: U13.37, U14.37
- new net GP182_PWM5: U17.37, U18.37
- new net GP182_PWM6: U21.37, U22.37
- new net GP182_PWM7: U25.37, U26.37
- new net GP182_PWM8: U29.37, U30.37
- new net GP183_PWM1: U5.39, U6.39
- new net GP183_PWM2: U10.39, U9.39
- new net GP183_PWM4: U13.39, U14.39
- new net GP183_PWM5: U17.39, U18.39
- new net GP183_PWM6: U21.39, U22.39
- new net GP183_PWM7: U25.39, U26.39
- new net GP183_PWM8: U29.39, U30.39
- new net GP19: SJ39.2, U10.25, U9.25
- new net GP19_I2C_1_SCL1: SJ28.3, U5.41, U6.41
- new net GP19_I2C_1_SCL2: SJ45.3, U10.41, U9.41
- new net GP19_I2C_1_SCL3: SJ62.3, U13.41, U14.41
- new net GP19_I2C_1_SCL4: SJ79.3, U17.41, U18.41
- new net GP19_I2C_1_SCL5: SJ96.3, U21.41, U22.41
- new net GP19_I2C_1_SCL6: SJ113.3, U25.41, U26.41
- new net GP19_I2C_1_SCL7: SJ130.3, U29.41, U30.41
- new net GP2: U5.42, U6.42
- new net GP20: U10.24, U9.24
- new net GP20_I2C_1_SDA1: SJ27.3, U5.43, U6.43
- new net GP20_I2C_1_SDA2: SJ44.3, U10.43, U9.43
- new net GP20_I2C_1_SDA3: SJ61.3, U13.43, U14.43
- new net GP20_I2C_1_SDA4: SJ78.3, U17.43, U18.43
- new net GP20_I2C_1_SDA5: SJ95.3, U21.43, U22.43
- new net GP20_I2C_1_SDA6: SJ112.3, U25.43, U26.43
- new net GP20_I2C_1_SDA7: SJ129.3, U29.43, U30.43
- new net GP21: U13.48, U14.48
- new net GP22: U13.42, U14.42
- new net GP23: SJ60.2, U13.34, U14.34
- new net GP24: SJ59.2, U13.32, U14.32
- new net GP25: SJ58.2, U13.30, U14.30
- new net GP26: SJ57.2, U13.28, U14.28
- new net GP27: U13.26, U14.26
- new net GP27_I2C_6_SCL1: U5.45, U6.45
- new net GP27_I2C_6_SCL2: U10.45, U9.45
- new net GP27_I2C_6_SCL3: U13.45, U14.45
- new net GP27_I2C_6_SCL4: U17.45, U18.45
- new net GP27_I2C_6_SCL5: U21.45, U22.45
- new net GP27_I2C_6_SCL6: U25.45, U26.45
- new net GP27_I2C_6_SCL7: U29.45, U30.45
- new net GP28: SJ56.2, U13.25, U14.25
- new net GP28_I2C_6_SDA1: U5.47, U6.47
- new net GP28_I2C_6_SDA2: U10.47, U9.47
- new net GP28_I2C_6_SDA3: U13.47, U14.47
- new net GP28_I2C_6_SDA4: U17.47, U18.47
- new net GP28_I2C_6_SDA5: U21.47, U22.47
- new net GP28_I2C_6_SDA6: U25.47, U26.47
- new net GP28_I2C_6_SDA7: U29.47, U30.47
- new net GP29: U13.24, U14.24
- new net GP3: SJ26.2, U5.34, U6.34
- new net GP30: U17.48, U18.48
- new net GP31: U17.42, U18.42
- new net GP32: SJ77.2, U17.34, U18.34
- new net GP33: SJ76.2, U17.32, U18.32
- new net GP34: SJ75.2, U17.30, U18.30
- new net GP35: SJ74.2, U17.28, U18.28
- new net GP36: U17.26, U18.26
- new net GP37: SJ73.2, U17.25, U18.25
- new net GP38: U17.24, U18.24
- new net GP39: U21.48, U22.48
- new net GP4: SJ25.2, U5.32, U6.32
- new net GP40: U21.42, U22.42
- new net GP40_I2S_2_CLK1: U5.52, U6.52
- new net GP40_I2S_2_CLK2: U10.52, U9.52
- new net GP40_I2S_2_CLK3: U13.52, U14.52
- new net GP40_I2S_2_CLK4: U17.52, U18.52
- new net GP40_I2S_2_CLK5: U21.52, U22.52
- new net GP40_I2S_2_CLK6: U25.52, U26.52
- new net GP40_I2S_2_CLK7: U29.52, U30.52
- new net GP41: SJ94.2, U21.34, U22.34
- new net GP41_I2S_2_FS1: U5.54, U6.54
- new net GP41_I2S_2_FS2: U10.54, U9.54
- new net GP41_I2S_2_FS3: U13.54, U14.54
- new net GP41_I2S_2_FS4: U17.54, U18.54
- new net GP41_I2S_2_FS5: U21.54, U22.54
- new net GP41_I2S_2_FS6: U25.54, U26.54
- new net GP41_I2S_2_FS7: U29.54, U30.54
- new net GP42: SJ93.2, U21.32, U22.32
- new net GP42_I2S_2_RXD1: U5.50, U6.50
- new net GP42_I2S_2_RXD2: U10.50, U9.50
- new net GP42_I2S_2_RXD3: U13.50, U14.50
- new net GP42_I2S_2_RXD4: U17.50, U18.50
- new net GP42_I2S_2_RXD5: U21.50, U22.50
- new net GP42_I2S_2_RXD6: U25.50, U26.50
- new net GP42_I2S_2_RXD7: U29.50, U30.50
- new net GP43: SJ92.2, U21.30, U22.30
- new net GP43_I2S_2_TXD1: U5.56, U6.56
- new net GP43_I2S_2_TXD2: U10.56, U9.56
- new net GP43_I2S_2_TXD3: U13.56, U14.56
- new net GP43_I2S_2_TXD4: U17.56, U18.56
- new net GP43_I2S_2_TXD5: U21.56, U22.56
- new net GP43_I2S_2_TXD6: U25.56, U26.56
- new net GP43_I2S_2_TXD7: U29.56, U30.56
- new net GP5: SJ24.2, U5.30, U6.30
- new net GP50: SJ91.2, U21.28, U22.28
- new net GP51: U21.26, U22.26
- new net GP52: SJ90.2, U21.25, U22.25
- new net GP53: U21.24, U22.24
- new net GP54: U25.48, U26.48
- new net GP55: U25.42, U26.42
- new net GP56: SJ111.2, U25.34, U26.34
- new net GP57: SJ110.2, U25.32, U26.32
- new net GP58: SJ109.2, U25.30, U26.30
- new net GP59: SJ108.2, U25.28, U26.28
- new net GP6: SJ23.2, U5.28, U6.28
- new net GP60: U25.26, U26.26
- new net GP61: SJ107.2, U25.25, U26.25
- new net GP62: U25.24, U26.24
- new net GP63: U29.48, U30.48
- new net GP64: U29.42, U30.42
- new net GP65: SJ128.2, U29.34, U30.34
- new net GP66: SJ127.2, U29.32, U30.32
- new net GP67: SJ126.2, U29.30, U30.30
- new net GP68: SJ125.2, U29.28, U30.28
- new net GP69: U29.26, U30.26
- new net GP7: U5.26, U6.26
- new net GP70: SJ124.2, U29.25, U30.25
- new net GP71: U29.24, U30.24
- new net GP77_SD_0_CD#1: U5.60, U6.60
- new net GP77_SD_0_CD#2: U10.60, U9.60
- new net GP77_SD_0_CD#3: U13.60, U14.60
- new net GP77_SD_0_CD#4: U17.60, U18.60
- new net GP77_SD_0_CD#5: U21.60, U22.60
- new net GP77_SD_0_CD#6: U25.60, U26.60
- new net GP77_SD_0_CD#7: U29.60, U30.60
- new net GP78_SD_0_CLK1: U5.58, U6.58
- new net GP78_SD_0_CLK2: U10.58, U9.58
- new net GP78_SD_0_CLK3: U13.58, U14.58
- new net GP78_SD_0_CLK4: U17.58, U18.58
- new net GP78_SD_0_CLK5: U21.58, U22.58
- new net GP78_SD_0_CLK6: U25.58, U26.58
- new net GP78_SD_0_CLK7: U29.58, U30.58
- new net GP79_SD_0_CMD1: U5.62, U6.62
- new net GP79_SD_0_CMD2: U10.62, U9.62
- new net GP79_SD_0_CMD3: U13.62, U14.62
- new net GP79_SD_0_CMD4: U17.62, U18.62
- new net GP79_SD_0_CMD5: U21.62, U22.62
- new net GP79_SD_0_CMD6: U25.62, U26.62
- new net GP79_SD_0_CMD7: U29.62, U30.62
- new net GP8: SJ22.2, U5.25, U6.25
- new net GP80_SD_0_DAT1: U5.66, U6.66
- new net GP80_SD_0_DAT2: U10.66, U9.66
- new net GP80_SD_0_DAT3: U13.66, U14.66
- new net GP80_SD_0_DAT4: U17.66, U18.66
- new net GP80_SD_0_DAT5: U21.66, U22.66
- new net GP80_SD_0_DAT6: U25.66, U26.66
- new net GP80_SD_0_DAT7: U29.66, U30.66
- new net GP81_SD_0_DAT2: U5.70, U6.70
- new net GP81_SD_0_DAT3: U10.70, U9.70
- new net GP81_SD_0_DAT4: U13.70, U14.70
- new net GP81_SD_0_DAT5: U17.70, U18.70
- new net GP81_SD_0_DAT6: U21.70, U22.70
- new net GP81_SD_0_DAT7: U25.70, U26.70
- new net GP81_SD_0_DAT8: U29.70, U30.70
- new net GP82_SD_0_DAT1: U5.64, U6.64
- new net GP82_SD_0_DAT3: U10.64, U9.64
- new net GP82_SD_0_DAT4: U13.64, U14.64
- new net GP82_SD_0_DAT5: U17.64, U18.64
- new net GP82_SD_0_DAT6: U21.64, U22.64
- new net GP82_SD_0_DAT7: U25.64, U26.64
- new net GP82_SD_0_DAT8: U29.64, U30.64
- new net GP83_SD_0_DAT1: U5.68, U6.68
- new net GP83_SD_0_DAT2: U10.68, U9.68
- new net GP83_SD_0_DAT4: U13.68, U14.68
- new net GP83_SD_0_DAT5: U17.68, U18.68
- new net GP83_SD_0_DAT6: U21.68, U22.68
- new net GP83_SD_0_DAT7: U25.68, U26.68
- new net GP83_SD_0_DAT8: U29.68, U30.68
- new net GP84_SD_CLK_FB1: U5.44, U6.44
- new net GP84_SD_CLK_FB2: U10.44, U9.44
- new net GP84_SD_CLK_FB3: U13.44, U14.44
- new net GP84_SD_CLK_FB4: U17.44, U18.44
- new net GP84_SD_CLK_FB5: U21.44, U22.44
- new net GP84_SD_CLK_FB6: U25.44, U26.44
- new net GP84_SD_CLK_FB7: U29.44, U30.44
- new net GP9: U5.24, U6.24
- new net INT1_XM1: SJ25.1, U7.13
- new net INT1_XM2: SJ42.1, U11.13
- new net INT1_XM3: SJ59.1, U15.13
- new net INT1_XM4: SJ76.1, U19.13
- new net INT1_XM5: SJ93.1, U23.13
- new net INT1_XM6: SJ110.1, U27.13
- new net INT1_XM7: SJ127.1, U31.13
- new net INT2_XM1: SJ26.1, U7.14
- new net INT2_XM2: SJ43.1, U11.14
- new net INT2_XM3: SJ60.1, U15.14
- new net INT2_XM4: SJ77.1, U19.14
- new net INT2_XM5: SJ94.1, U23.14
- new net INT2_XM6: SJ111.1, U27.14
- new net INT2_XM7: SJ128.1, U31.14
- new net INT_G1: SJ23.1, U7.11
- new net INT_G2: SJ40.1, U11.11
- new net INT_G3: SJ57.1, U15.11
- new net INT_G4: SJ74.1, U19.11
- new net INT_G5: SJ91.1, U23.11
- new net INT_G6: SJ108.1, U27.11
- new net INT_G7: SJ125.1, U31.11
- new net MSIC_SLP_CLK1: U5.7, U6.7
- new net MSIC_SLP_CLK2: U10.7, U9.7
- new net MSIC_SLP_CLK3: U13.7, U14.7
- new net MSIC_SLP_CLK4: U17.7, U18.7
- new net MSIC_SLP_CLK5: U21.7, U22.7
- new net MSIC_SLP_CLK6: U25.7, U26.7
- new net MSIC_SLP_CLK7: U29.7, U30.7
- new net N$10: C8.1, U7.7
- new net N$11: R7.2, SJ30.3
- new net N$14: R8.2, SJ30.1
- new net N$15: R9.2, SJ29.1
- new net N$16: R10.2, SJ29.3
- new net N$17: R11.2, SJ31.1
- new net N$18: R12.2, SJ32.1
- new net N$19: C13.1, U11.9
- new net N$20: C13.2, U11.8
- new net N$21: C14.1, U11.7
- new net N$22: R13.2, SJ47.3
- new net N$23: R14.2, SJ47.1
- new net N$24: R15.2, SJ46.1
- new net N$25: R16.2, SJ46.3
- new net N$26: R17.2, SJ48.1
- new net N$27: R18.2, SJ49.1
- new net N$28: C19.1, U15.9
- new net N$29: C19.2, U15.8
- new net N$30: C20.1, U15.7
- new net N$31: R19.2, SJ64.3
- new net N$32: R20.2, SJ64.1
- new net N$33: R21.2, SJ63.1
- new net N$34: R22.2, SJ63.3
- new net N$35: R23.2, SJ65.1
- new net N$36: R24.2, SJ66.1
- new net N$37: C25.1, U19.9
- new net N$38: C25.2, U19.8
- new net N$39: C26.1, U19.7
- new net N$40: R25.2, SJ81.3
- new net N$41: R26.2, SJ81.1
- new net N$42: R27.2, SJ80.1
- new net N$43: R28.2, SJ80.3
- new net N$44: R29.2, SJ82.1
- new net N$45: R30.2, SJ83.1
- new net N$46: C31.1, U23.9
- new net N$47: C31.2, U23.8
- new net N$48: C32.1, U23.7
- new net N$49: R31.2, SJ98.3
- new net N$50: R32.2, SJ98.1
- new net N$51: R33.2, SJ97.1
- new net N$52: R34.2, SJ97.3
- new net N$53: R35.2, SJ99.1
- new net N$54: R36.2, SJ100.1
- new net N$55: C37.1, U27.9
- new net N$56: C37.2, U27.8
- new net N$57: C38.1, U27.7
- new net N$58: R37.2, SJ115.3
- new net N$59: R38.2, SJ115.1
- new net N$60: R39.2, SJ114.1
- new net N$61: R40.2, SJ114.3
- new net N$62: R41.2, SJ116.1
- new net N$63: R42.2, SJ117.1
- new net N$64: C43.1, U31.9
- new net N$65: C43.2, U31.8
- new net N$66: C44.1, U31.7
- new net N$67: R43.2, SJ132.3
- new net N$68: R44.2, SJ132.1
- new net N$69: R45.2, SJ131.1
- new net N$70: R46.2, SJ131.3
- new net N$71: R47.2, SJ133.1
- new net N$72: R48.2, SJ134.1
- new net N$8: C7.1, U7.9
- new net N$9: C7.2, U7.8
- new net OSC_CLK_OUT1: U5.67, U6.67
- new net OSC_CLK_OUT2: U10.67, U9.67
- new net OSC_CLK_OUT3: U13.67, U14.67
- new net OSC_CLK_OUT4: U17.67, U18.67
- new net OSC_CLK_OUT5: U21.67, U22.67
- new net OSC_CLK_OUT6: U25.67, U26.67
- new net OSC_CLK_OUT7: U29.67, U30.67
- new net PSW1: U5.21, U6.21
- new net PSW2: U10.21, U9.21
- new net PSW3: U13.21, U14.21
- new net PSW4: U17.21, U18.21
- new net PSW5: U21.21, U22.21
- new net PSW6: U25.21, U26.21
- new net PSW7: U29.21, U30.21
- new net PWRBTN#1: U5.17, U6.17
- new net PWRBTN#2: U10.17, U9.17
- new net PWRBTN#3: U13.17, U14.17
- new net PWRBTN#4: U17.17, U18.17
- new net PWRBTN#5: U21.17, U22.17
- new net PWRBTN#6: U25.17, U26.17
- new net PWRBTN#7: U29.17, U30.17
- new net RCVR_MODE1: U5.31, U6.31
- new net RCVR_MODE2: U10.31, U9.31
- new net RCVR_MODE3: U13.31, U14.31
- new net RCVR_MODE4: U17.31, U18.31
- new net RCVR_MODE5: U21.31, U22.31
- new net RCVR_MODE6: U25.31, U26.31
- new net RCVR_MODE7: U29.31, U30.31
- new net RESET_OUT#1: U5.36, U6.36
- new net RESET_OUT#2: U10.36, U9.36
- new net RESET_OUT#3: U13.36, U14.36
- new net RESET_OUT#4: U17.36, U18.36
- new net RESET_OUT#5: U21.36, U22.36
- new net RESET_OUT#6: U25.36, U26.36
- new net RESET_OUT#7: U29.36, U30.36
- new net SCL1: R8.1, SJ28.2, U7.21
- new net SCL2: R14.1, SJ45.2, U11.21
- new net SCL3: R20.1, SJ62.2, U15.21
- new net SCL4: R26.1, SJ79.2, U19.21
- new net SCL5: R32.1, SJ96.2, U23.21
- new net SCL6: R38.1, SJ113.2, U27.21
- new net SCL7: R44.1, SJ130.2, U31.21
- new net SDA1: R7.1, SJ27.2, U7.24
- new net SDA2: R13.1, SJ44.2, U11.24
- new net SDA3: R19.1, SJ61.2, U15.24
- new net SDA4: R25.1, SJ78.2, U19.24
- new net SDA5: R31.1, SJ95.2, U23.24
- new net SDA6: R37.1, SJ112.2, U27.24
- new net SDA7: R43.1, SJ129.2, U31.24
- new net SDO_G1: R12.1, SJ20.1, SJ34.2, U7.22
- new net SDO_G2: R18.1, SJ37.1, SJ51.2, U11.22
- new net SDO_G3: R24.1, SJ54.1, SJ68.2, U15.22
- new net SDO_G4: R30.1, SJ71.1, SJ85.2, U19.22
- new net SDO_G5: R36.1, SJ102.2, SJ88.1, U23.22
- new net SDO_G6: R42.1, SJ105.1, SJ119.2, U27.22
- new net SDO_G7: R48.1, SJ122.1, SJ136.2, U31.22
- new net SDO_XM1: R11.1, SJ21.1, SJ33.2, U7.23
- new net SDO_XM2: R17.1, SJ38.1, SJ50.2, U11.23
- new net SDO_XM3: R23.1, SJ55.1, SJ67.2, U15.23
- new net SDO_XM4: R29.1, SJ72.1, SJ84.2, U19.23
- new net SDO_XM5: R35.1, SJ101.2, SJ89.1, U23.23
- new net SDO_XM6: R41.1, SJ106.1, SJ118.2, U27.23
- new net SDO_XM7: R47.1, SJ123.1, SJ135.2, U31.23
- new net USB_DN1: U5.18, U6.18
- new net USB_DN2: U10.18, U9.18
- new net USB_DN3: U13.18, U14.18
- new net USB_DN4: U17.18, U18.18
- new net USB_DN5: U21.18, U22.18
- new net USB_DN6: U25.18, U26.18
- new net USB_DN7: U29.18, U30.18
- new net USB_DP1: U5.16, U6.16
- new net USB_DP2: U10.16, U9.16
- new net USB_DP3: U13.16, U14.16
- new net USB_DP4: U17.16, U18.16
- new net USB_DP5: U21.16, U22.16
- new net USB_DP6: U25.16, U26.16
- new net USB_DP7: U29.16, U30.16
- new net USB_ID1: U5.3, U6.3
- new net USB_ID2: U10.3, U9.3
- new net USB_ID3: U13.3, U14.3
- new net USB_ID4: U17.3, U18.3
- new net USB_ID5: U21.3, U22.3
- new net USB_ID6: U25.3, U26.3
- new net USB_ID7: U29.3, U30.3
- new net USB_VBUS1: U5.20, U6.20
- new net USB_VBUS2: U10.20, U9.20
- new net USB_VBUS3: U13.20, U14.20
- new net USB_VBUS4: U17.20, U18.20
- new net USB_VBUS5: U21.20, U22.20
- new net USB_VBUS6: U25.20, U26.20
- new net USB_VBUS7: U29.20, U30.20
- new net VSYS1: C11.1, U5.2, U5.4, U5.6, U6.2, U6.4, U6.6, U8.1, U8.3
- new net VSYS2: C17.1, U10.2, U10.4, U10.6, U12.1, U12.3, U9.2, U9.4, U9.6
- new net VSYS3: C23.1, U13.2, U13.4, U13.6, U14.2, U14.4, U14.6, U16.1, U16.3
- new net VSYS4: C29.1, U17.2, U17.4, U17.6, U18.2, U18.4, U18.6, U20.1, U20.3
- new net VSYS5: C35.1, U21.2, U21.4, U21.6, U22.2, U22.4, U22.6, U24.1, U24.3
- new net VSYS6: C41.1, U25.2, U25.4, U25.6, U26.2, U26.4, U26.6, U28.1, U28.3
- new net VSYS7: C47.1, U29.2, U29.4, U29.6, U30.2, U30.4, U30.6, U32.1, U32.3
- new net V_BAT_BKUP1: U5.23, U6.23
- new net V_BAT_BKUP2: U10.23, U9.23
- new net V_BAT_BKUP3: U13.23, U14.23
- new net V_BAT_BKUP4: U17.23, U18.23
- new net V_BAT_BKUP5: U21.23, U22.23
- new net V_BAT_BKUP6: U25.23, U26.23
- new net V_BAT_BKUP7: U29.23, U30.23
Routing:
- net GP43: track 0.00 -> 72.4 mm, vias 0 -> 3
- net GP34: track 0.00 -> 72.4 mm, vias 0 -> 3
- net GP67: track 0.00 -> 72.4 mm, vias 0 -> 3
- net GP58: track 0.00 -> 72.4 mm, vias 0 -> 3
- net GP5: track 0.00 -> 72.4 mm, vias 0 -> 3
- net GP25: track 0.00 -> 72.4 mm, vias 0 -> 3
- net GP16: track 0.00 -> 72.4 mm, vias 0 -> 3
- net GP33: track 0.00 -> 64.1 mm, vias 0 -> 3
- net GP66: track 0.00 -> 64.1 mm, vias 0 -> 3
- net GP57: track 0.00 -> 64.1 mm, vias 0 -> 3
- net GP42: track 0.00 -> 64.1 mm, vias 0 -> 3
- net GP4: track 0.00 -> 64.1 mm, vias 0 -> 3
- net GP24: track 0.00 -> 64.1 mm, vias 0 -> 3
- net GP13: track 0.00 -> 64.1 mm, vias 0 -> 3
- net GP109_SPI_2_CLK4: track 0.00 -> 62.1 mm, vias 0 -> 2
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- added copper zone on layer 1, net 3.3V_LOCAL1
- added copper zone on layer 1, net 3.3V_LOCAL2
- added copper zone on layer 1, net 3.3V_LOCAL3
- added copper zone on layer 1, net 3.3V_LOCAL4
- added copper zone on layer 1, net 3.3V_LOCAL5
- added copper zone on layer 1, net 3.3V_LOCAL6
- added copper zone on layer 1, net 3.3V_LOCAL7
- added copper zone on layer 1, net GND1
- added copper zone on layer 16, net GND1
- added copper zone on layer 1, net GND2
- added copper zone on layer 16, net GND2
- added copper zone on layer 1, net GND3
- added copper zone on layer 16, net GND3
- added copper zone on layer 1, net GND4
- added copper zone on layer 16, net GND4
- added copper zone on layer 1, net GND5
- added copper zone on layer 16, net GND5
- added copper zone on layer 1, net GND6
- added copper zone on layer 16, net GND6
- added copper zone on layer 1, net GND7
- added copper zone on layer 16, net GND7
Other:
- board size 30.5 x 44.5 mm -> 137.2 x 103.1 mm
